Commit message: 补交代码

File: nav_ws/src/mysystem/urdf/robot.urdf (robot description, URDF)
Before this commit: robot robot, 9 links, 8 joints
Links:
- removed link imu
- removed link livox_frame
- added link aft_mapped, mass 0.33968131; collision mesh filename=package://mysystem/meshes/livox_frame.stl; visual mesh filename=package://mysystem/meshes/livox_frame.stl
Joints:
- removed joint joint_imu_up
- removed joint joint_livox_frame
- added joint joint_aft_mapped: type fixed, parent up, child aft_mapped, origin xyz=-0.0808 0 0.0951 rpy=0.0000103944 0.78539265 -3.1415853037
- joint joint_up: origin xyz=0 0 0.1039 rpy=0 0 0 -> xyz=0 0 0.1039 rpy=0 0 3.141592653589793
